Commit message: initial commit

File: eufs_description/robots/ads-dv.urdf.xacro (robot description, xacro)
@@ -1,36 +1,14 @@
 <?xml version="1.0"?>
 <robot name="eufs" xmlns:xacro="http://www.ros.org/wiki/xacro">
-    <!-- ***************** -->
-    <!-- Imported elements -->
-    <!-- ***************** -->
-    <!-- First we import all posible elements defined in the urdf.xacro files. All these elements are defined as macro:xacros -->
-    <!-- Import Robotnik CAR base elements -->
     <xacro:include filename="$(find eufs_description)/urdf/bases/ads-dv_base.urdf.xacro" />
-    <!-- Import Robotnik CAR wheels -->
     <xacro:include filename="$(find eufs_description)/urdf/wheels/suspension_wheel.urdf.xacro" />
-    <!-- Import all available sensors -->
     <xacro:include filename="$(find eufs_description)/sensors/all_sensors.urdf.xacro" />
-    <!-- ***************** -->
-    <!-- Global parameters -->
-    <!-- ***************** -->
     <xacro:property name="PI" value="3.1415926535897931"/>
-    <!-- Wheel parameters -->
-    <xacro:property name="wheel_offset_x" value="1.0" />    <!-- x,y,z in translation from base_link to the center of the wheel -->
+    <xacro:property name="wheel_offset_x" value="1.0" />
     <xacro:property name="wheel_offset_y" value="0.75" />
     <xacro:property name="wheel_offset_z" value="0.0" />
-    <!-- Flag to select the high or low quality model -->
     <xacro:property name="hq" value="true" />
-    <!-- *************** -->
-    <!-- Robots Elements -->
-    <!-- *************** -->
-    <!-- Here we create the robot elements using the xacro:macros imported at the beggining of this file -->
-    <!-- Summit XL base -->
     <xacro:eufs_base name="eufs" publish_bf="true" hq="${hq}" />
-    <!-- Gazebo ros control pluggins -->
     <xacro:ros_control/>
-    <!-- Gazebo skid steering pluggins -->
-    <!-- xacro:skid_steering broadcastOdomTF="1"/ -->
-    <!-- WHEELS -->
-    <!-- Wheels -->
     <xacro:front_wheel lr_prefix="left" fr_prefix="front"
         lr_reflect="1" fr_reflect="1"/>
@@ -41,53 +19,6 @@
     <xacro:rear_wheel lr_prefix="right" fr_prefix="rear"
         lr_reflect="-1" fr_reflect="-1"/>
-    <!-- MAIN SENSORS -->
-<!--     LOCATIONS: (XYZ)
-    IMU: 0.0 0.0 0.170
-    GPS: -0.110 0.0 0.9
-    LIDAR: 1.700 0.0 -0.150
-    STEREO CAM: -0.110 0.0 0.800 -->
-    <xacro:sensor_imu parent="base_link" prefix="imu">
-        <origin xyz="-0.0 0.0 0.0" rpy="0 0 0"/>
-    </xacro:sensor_imu>
-    <xacro:sensor_gps  parent="base_link" prefix="gps">
-        <origin xyz="0.0 0.0 0.4" rpy="0 0 0"/>
-    </xacro:sensor_gps>
-<!--     <xacro:sensor_hokuyo_utm30lx  parent="base_link" prefix="lidar" >
-        <origin xyz="1.700 0.0 -0.080" rpy="0 -0.0174533 0"/>
-    </xacro:sensor_hokuyo_utm30lx> -->
-    <!-- <xacro:VLP-16  parent="base_link" name="velodyne" topic="/velodyne_points" hz="10">
+     <xacro:VLP-16  parent="base_link" name="velodyne" topic="/velodyne_points" hz="10">
         <origin xyz="1.700 0.0 -0.150" rpy="0 -0.0174533 0"/>
-    </xacro:VLP-16> -->
-    <xacro:VLP-16R  parent="base_link" name="velodyne" topic="/velodyne_points" hz="10" samples="800">
-        <origin xyz="1.58 0.0 -0.1" rpy="0 ${1*M_PI/180.0} 0"/>
-    </xacro:VLP-16R>
-    <xacro:zed_camera parent="base_link" prefix="zed">
-        <origin xyz="0.1 0.0 0.52" rpy="0 0 0"/>
-    </xacro:zed_camera>
-    <!-- EXTRA SENSORS FROM THE ROBOTNIK SENSORS LIBRARY -->
-<!--
-    <xacro:sensor_hokuyo3d name="hokuyo3d" parent="base_link">
-        <origin xyz="0.9 0.0 0.450" rpy="0 0.35 0"/>
-    </xacro:sensor_hokuyo3d>
-    <xacro:sensor_hokuyo_urg04lx name="hokuyo1" parent="base_link">
-        <origin xyz="-0.1 0.0 0.33" rpy="0 0 0"/>
-    </xacro:sensor_hokuyo_urg04lx>
-    <xacro:sensor_axis name="camera" parent="base_link">
-        <origin xyz="0.19 0 0.17" rpy="0 ${15*PI/180} 0"/>
-    </xacro:sensor_axis>
-    <xacro:sensor_asus_xtion_pro name="xtion_pro" parent="base_link">
-        <origin xyz="0.3 0.0 0.3" rpy="0 0 0"/>
-    </xacro:sensor_asus_xtion_pro>
-    <xacro:sensor_kinect parent="base_link" prefix="kinect">
-        <origin xyz="0.0 0.0 0.45" rpy="0 0 0"/>
-    </xacro:sensor_kinect>
-    <xacro:BB2-08S2C-60  prefix="bee" frame="bee" name="bee"/>
-    <xacro:sensor_fotonic name="fotonic" parent="base_link">
-        <origin xyz="0.3 0.0 0.24" rpy="0 0 0"/>
-    </xacro:sensor_fotonic>   -->
-    <!-- PLUGINS -->
-    <!-- ros control plugin -->
-<!--   <gazebo>
-    <plugin name="gazebo_ros_control" filename="libgazebo_ros_control.so"/>
-</gazebo> -->
+    </xacro:VLP-16>
 </robot>

File: eufs_description/robots/eufs.urdf.xacro (robot description, xacro)
@@ -41,10 +41,10 @@
         lr_reflect="-1" fr_reflect="-1"/>
     <!-- MAIN SENSORS -->
-    <xacro:sensor_imu parent="base_link" prefix="imu">
+    <!-- <xacro:sensor_imu parent="base_link" prefix="imu">
         <origin xyz="0.0 0.0 0.170" rpy="0 0 0"/>
     </xacro:sensor_imu>
     <xacro:sensor_gps  parent="base_link" prefix="gps">
         <origin xyz="-0.110 0.0 0.9" rpy="0 0 0"/>
-    </xacro:sensor_gps>
+    </xacro:sensor_gps> -->
 <!--     <xacro:sensor_hokuyo_utm30lx  parent="base_link" prefix="lidar" >
         <origin xyz="1.700 0.0 -0.080" rpy="0 -0.0174533 0"/>
@@ -56,7 +56,7 @@
         <origin xyz="1.700 0.0 -0.150" rpy="0 -${1.5*M_PI/180.0} 0"/>
     </xacro:VLP-16>
-    <xacro:zed_camera parent="base_link" prefix="zed">
+    <!-- <xacro:zed_camera parent="base_link" prefix="zed">
         <origin xyz="-0.110 0.0 0.84" rpy="0 0 0"/>
-    </xacro:zed_camera>
+    </xacro:zed_camera>   -->
     <!-- EXTRA SENSORS FROM THE ROBOTNIK SENSORS LIBRARY -->
 <!--

File: eufs_description/sensors/VLP-16.urdf.xacro (robot description, xacro)
@@ -2,5 +2,5 @@
 <robot xmlns:xacro="http://www.ros.org/wiki/xacro" name="VLP-16">
   <xacro:property name="M_PI" value="3.1415926535897931" />
-  <xacro:macro name="VLP-16" params="*origin parent:=base_link name:=velodyne topic:=/velodyne_points hz:=10 lasers:=16 samples:=1875 collision_range:=0.3 min_range:=0.9 max_range:=130.0 noise:=0.008 min_angle:=-${M_PI} max_angle:=${M_PI}">
+  <xacro:macro name="VLP-16" params="*origin parent:=base_link name:=velodyne topic:=/velodyne_points hz:=10 lasers:=16 samples:=2000 collision_range:=0.3 min_range:=0.9 max_range:=130.0 noise:=0.008 min_angle:=-${M_PI} max_angle:=${M_PI}">
     <joint name="${name}_base_mount_joint" type="fixed">
       <xacro:insert_block name="origin" />

File: eufs_description/sensors/all_sensors.urdf.xacro (robot description, xacro)
@@ -1,23 +1,5 @@
 <?xml version="1.0"?>
 <robot name="all_sensors" xmlns:xacro="http://www.ros.org/wiki/xacro">
-  <!-- This file unifies all sensors that can be used on simulation, defined as xacro:macros -->
-  <!-- GPS -->
-  <xacro:include filename="$(find eufs_description)/sensors/gps.urdf.xacro"/>
-  <!-- Hokuyo utm30lx -->
-  <xacro:include filename="$(find eufs_description)/sensors/hokuyo_utm30lx.urdf.xacro"/>
-  <!-- Velodyne VLP-16 -->
+  This file unifies all sensors that can be used on simulation, defined as xacro:macros
   <xacro:include filename="$(find eufs_description)/sensors/VLP-16.urdf.xacro"/>
-  <xacro:include filename="$(find eufs_description)/sensors/VLP-16R.urdf.xacro"/>
-  <!-- Imu -->
-  <xacro:include filename="$(find eufs_description)/sensors/imu.urdf.xacro"/>
-  <!-- Imu hector -->
-  <xacro:include filename="$(find eufs_description)/sensors/imu_hector_plugin.urdf.xacro"/>
-  <!-- Kinect -->
-  <xacro:include filename="$(find eufs_description)/sensors/kinect.urdf.xacro"/>
-  <!-- KinectV2 -->
-  <xacro:include filename="$(find eufs_description)/sensors/kinectv2.urdf.xacro"/>
-  <!-- Pointgrey Bumblebee -->
-  <xacro:include filename="$(find eufs_description)/sensors/pointgrey_bumblebee2.urdf.xacro"/>
-  <!-- ZED Stereo camera -->
-  <xacro:include filename="$(find eufs_description)/sensors/zed.urdf.xarco"/>
-</robot>
+  </robot>
